Commit message: Add switch for GPU laser Gazebo plugin

File: amiro_description/urdf/amiro_camera_hokuyo.xacro (robot description, xacro)
@@ -9,5 +9,5 @@
   <!-- Laser -->
   <xacro:include filename="$(find amiro_description)/urdf/laser/hokuyo.xacro"/>
-  <xacro:laser name="laser" parent="${base_link}" xyz="0 0 ${hokuyo_link_height}" rpy="0 ${hokuyo_base_pitch} 0" meshes="package://amiro_description/meshes/laser"/>
+  <xacro:laser name="laser" parent="${base_link}" xyz="0 0 ${hokuyo_link_height}" rpy="0 ${hokuyo_base_pitch} 0" meshes="package://amiro_description/meshes/laser" use_gpu="$(arg use_gpu_laser)" />
   <!-- Camera -->
   <xacro:include filename="$(find amiro_description)/urdf/camera/camera.xacro"/>

File: amiro_description/urdf/amiro_hokuyo.xacro (robot description, xacro)
@@ -9,4 +9,4 @@
   <!-- Laser -->
   <xacro:include filename="$(find amiro_description)/urdf/laser/hokuyo.xacro"/>
-  <xacro:laser name="laser" parent="${base_link}" xyz="0 0 ${hokuyo_link_height}" rpy="0 ${hokuyo_base_pitch} 0" meshes="package://amiro_description/meshes/laser"/>
+  <xacro:laser name="laser" parent="${base_link}" xyz="0 0 ${hokuyo_link_height}" rpy="0 ${hokuyo_base_pitch} 0" meshes="package://amiro_description/meshes/laser" use_gpu="$(arg use_gpu_laser)" />
 </robot>

File: amiro_description/urdf/laser/hokuyo.xacro (robot description, xacro)
@@ -1,9 +1,17 @@
 <?xml version="1.0"?>
 <robot xmlns:xacro="http://www.ros.org/wiki/xacro">
-<xacro:macro name="laser" params="name parent xyz rpy meshes" >
+<xacro:macro name="laser" params="name parent xyz rpy meshes use_gpu:=false" >
   <xacro:property name="base_width" value="0.05" /> <!-- (m) base width of housing -->
   <xacro:property name="base_depth" value="0.05" /> <!-- (m) base depth of housing -->
   <xacro:property name="base_height" value="0.07" /> <!-- (m) base heigth of housing -->
   <xacro:property name="laser_height" value="${base_height / 2 + 0.02275}" /> <!-- (m) origin of the laser measurement -->
+  <xacro:if value="${use_gpu}">
+    <xacro:property name="sensor_type" value="gpu_ray" />
+    <xacro:property name="plugin_name" value="libgazebo_ros_gpu_laser.so" />
+  </xacro:if>
+  <xacro:unless value="${use_gpu}">
+    <xacro:property name="sensor_type" value="ray" />
+    <xacro:property name="plugin_name" value="libgazebo_ros_laser.so" />
+  </xacro:unless>
   <joint name="${parent}_${name}_base_joint" type="fixed">
     <axis xyz="0 0 1" />
@@ -40,5 +48,5 @@
   </link>
     <gazebo reference="${name}">
-        <sensor name="laser" type="ray">
+        <sensor name="laser" type="${sensor_type}">
         <pose>0 0 0 0 0 0</pose>
           <ray>
@@ -58,5 +66,5 @@
             </range>
           </ray>
-          <plugin name="laser" filename="libgazebo_ros_laser.so" >
+          <plugin name="laser" filename="${plugin_name}" >
             <robotNamespace></robotNamespace>
             <topicName>${name}/scan</topicName>
