Commit message: Update AMiRo model (still not original) with diff. drive. Now using namespace with example of amiro1 in 'roslaunch amiro_gazebo amiro_world.launch'
Signed-off-by: Timo Korthals <tkorthals@cit-ec.uni-bielefeld.de>

File: amiro_description/urdf/amiro.xacro (robot description, xacro)
@@ -12,49 +12,23 @@
   <xacro:property name="wheel_dia" value="0.05571" /> <!-- amiro wheel diameter -->
   <xacro:property name="wheel_mass" value="0.02" /> <!-- amiro wheel diameter -->
-  <xacro:property name="base_link_height" value="0.045" /> <!-- amiro base link height -->
-  <xacro:property name="base_link" value="base_link" /> <!-- amiro base link -->
-  <xacro:property name="left_wheel_link" value="left_wheel_link" /> <!-- amiro wheel link -->
-  <xacro:property name="right_wheel_link" value="right_wheel_link" /> <!-- amiro wheel link -->
+  <xacro:property name="base_link_clearance" value="0.0026" /> <!-- space between floor and amiro base -->
+  <xacro:property name="base_link_height" value="${base_link_clearance + height / 2}" /> <!-- amiro base link height -->
+  <xacro:property name="prefix" value="" /> <!--""-->
+  <xacro:property name="base_link" value="${prefix}base_link" /> <!-- amiro base link -->
+  <xacro:property name="left_wheel_link" value="${prefix}left_wheel_link" /> <!-- amiro wheel link -->
+  <xacro:property name="right_wheel_link" value="${prefix}right_wheel_link" /> <!-- amiro wheel link -->
+  <xacro:property name="right_wheel_joint" value="${prefix}right_wheel_joint" /> <!-- amiro wheel joint -->
+  <xacro:property name="left_wheel_joint" value="${prefix}left_wheel_joint" /> <!-- amiro wheel joint -->
+  <xacro:property name="odom" value="${prefix}odom" /> <!-- amiro odometry topic/tf -->
+  <xacro:property name="cmd_vel" value="${prefix}cmd_vel" /> <!-- amiro differential command  topic -->
+  <xacro:property name="update_rate" value="$(arg update_rate)" /> <!-- update rate for the plugins and TFs -->
   <!-- Import all Gazebo-customization elements, including Gazebo colors -->
   <xacro:include filename="$(find amiro_description)/urdf/amiro.gazebo" />
   <!-- Import Rviz colors -->
   <xacro:include filename="$(find amiro_description)/urdf/materials.xacro" />
-  <gazebo>
-    <!--<plugin filename="libgazebo_ros_control.so" name="ros_control">
-      <robotNamespace></robotNamespace>
-    </plugin>-->
-    <plugin name="differential_drive_controller" filename="libgazebo_ros_diff_drive.so">
-        <alwaysOn>true</alwaysOn>
-        <updateRate>50</updateRate>
-        <leftJoint>left_wheel_joint</leftJoint>
-        <rightJoint>right_wheel_joint</rightJoint>
-        <wheelSeparation>0.069</wheelSeparation> <!-- meter -->
-        <wheelDiameter>0.05571</wheelDiameter> <!-- meter -->
-        <wheelTorque>1</wheelTorque> <!-- Nm ? -->
-        <!--<odometrySource>1</odometrySource>--> <!-- ? -->
-        <commandTopic>cmd_vel</commandTopic>
-        <odometryTopic>odom</odometryTopic>
-        <odometryFrame>odom</odometryFrame>
-        <robotBaseFrame>base_link</robotBaseFrame>
-        <!--<publishTf>foo</publishTf>--> <!-- Use robot model name as prefix -->
-        <!--<robotNamespace>foo</robotNamespace>--> <!-- Use robot model name as namespace -->
-        <rosDebugLevel>2</rosDebugLevel>
-        <publishWheelTF>true</publishWheelTF>
-        <publishWheelJointState>true</publishWheelJointState>
-        <legacyMode>false</legacyMode>
-        <wheelAcceleration>1</wheelAcceleration> <!-- rad/s^2 -->
-        <wheelAcceleration>1</wheelAcceleration> <!-- rad/s^2 -->
-    </plugin>
-</gazebo>
-<!--   <xacro:macro name="amiro_body" params="parent"> -->
-  <!-- Used for fixing robot to Gazebo 'base_link' -->
-<!--   <link name="base_link"/> -->
-<!--  <joint name="fixed" type="fixed">
-    <parent link="world"/>
-    <child link="${base_link}"/>
-  </joint>-->
   <!-- Base Link -->
   <link name="${base_link}">
-    <collision>
+    <!-- Base -->
+    <collision name='base_collision'>
       <origin xyz="0 0 ${base_link_height}" rpy="0 0 0"/>
       <geometry>
@@ -62,5 +36,5 @@
       </geometry>
     </collision>
-    <visual>
+    <visual name='base_visual'>
       <origin xyz="0 0 ${base_link_height}" rpy="0 0 0"/>
       <geometry>
@@ -69,5 +43,5 @@
       <material name="orange"/>
     </visual>
-    <inertial>
+    <inertial name='base_inertia'>
       <origin xyz="0 0 ${base_link_height}" rpy="0 0 0"/>
       <mass value="${mass}"/>
@@ -77,7 +51,43 @@
         izz="0.005"/>
     </inertial>
+    <!-- Front caster -->
+    <collision name='caster_front_collision'>
+      <origin xyz="0.042 0 0.001" rpy="0 0 0"/>
+      <geometry>
+        <sphere radius="0.002"/>
+      </geometry>
+    </collision>
+    <visual name='caster_front_visual'>
+      <origin xyz="0.042 0 0.001" rpy="0 0 0"/>
+      <geometry>
+        <sphere radius="0.002"/>
+      </geometry>
+      <material name="orange"/>
+    </visual>
+    <inertial name='caster_front_inertia'>
+      <origin xyz="0.042 0 0.001" rpy="0 0 0"/>
+      <mass value="0.01"/>
+    </inertial>
+    <!-- Back caster -->
+    <collision name='caster_back_collision'>
+      <origin xyz="-0.042 0 0.001" rpy="0 0 0"/>
+      <geometry>
+        <sphere radius="0.002"/>
+      </geometry>
+    </collision>
+    <visual name='caster_back_visual'>
+      <origin xyz="-0.042 0 0.001" rpy="0 0 0"/>
+      <geometry>
+        <sphere radius="0.002"/>
+      </geometry>
+      <material name="orange"/>
+    </visual>
+    <inertial name='caster_back_inertia'>
+      <origin xyz="-0.042 0 0.001" rpy="0 0 0"/>
+      <mass value="0.01"/>
+    </inertial>
   </link>
   <!-- Left wheel -->
-  <joint name="left_wheel_joint" type="continuous">
+  <joint name="${left_wheel_joint}" type="continuous">
     <parent link="${base_link}"/>
     <child link="${left_wheel_link}"/>
@@ -110,5 +120,5 @@
   </link>
   <!-- Right wheel -->
-  <joint name="right_wheel_joint" type="continuous">
+  <joint name="${right_wheel_joint}" type="continuous">
     <parent link="${base_link}"/>
     <child link="${right_wheel_link}"/>
@@ -140,138 +150,3 @@
     </inertial>
   </link>
-<!--
-  <joint name="joint1" type="continuous">
-    <parent link="link1"/>
-    <child link="link2"/>
-    <origin xyz="0 ${width} ${height1 - axel_offset}" rpy="0 0 0"/>
-    <axis xyz="0 1 0"/>
-    <dynamics damping="0.7"/>
-  </joint>
-  Middle Link
-  <link name="link2">
-    <collision>
-      <origin xyz="0 0 ${height2/2 - axel_offset}" rpy="0 0 0"/>
-      <geometry>
-        <box size="${width} ${width} ${height2}"/>
-      </geometry>
-    </collision>
-    <visual>
-      <origin xyz="0 0 ${height2/2 - axel_offset}" rpy="0 0 0"/>
-      <geometry>
-        <box size="${width} ${width} ${height2}"/>
-      </geometry>
-      <material name="black"/>
-    </visual>
-    <inertial>
-      <origin xyz="0 0 ${height2/2 - axel_offset}" rpy="0 0 0"/>
-      <mass value="${mass}"/>
-      <inertia
-          ixx="${mass / 12.0 * (width*width + height2*height2)}" ixy="0.0" ixz="0.0"
-          iyy="${mass / 12.0 * (height2*height2 + width*width)}" iyz="0.0"
-          izz="${mass / 12.0 * (width*width + width*width)}"/>
-    </inertial>
-  </link>
-  <joint name="joint2" type="continuous">
-    <parent link="link2"/>
-    <child link="link3"/>
-    <origin xyz="0 ${width} ${height2 - axel_offset*2}" rpy="0 0 0"/>
-    <axis xyz="0 1 0"/>
-    <dynamics damping="0.7"/>
-  </joint>
-  Top Link
-  <link name="link3">
-    <collision>
-      <origin xyz="0 0 ${height3/2 - axel_offset}" rpy="0 0 0"/>
-      <geometry>
-        <box size="${width} ${width} ${height3}"/>
-      </geometry>
-    </collision>
-    <visual>
-      <origin xyz="0 0 ${height3/2 - axel_offset}" rpy="0 0 0"/>
-      <geometry>
-        <box size="${width} ${width} ${height3}"/>
-      </geometry>
-      <material name="orange"/>
-    </visual>
-    <inertial>
-      <origin xyz="0 0 ${height3/2 - axel_offset}" rpy="0 0 0"/>
-      <mass value="${mass}"/>
-      <inertia
-          ixx="${mass / 12.0 * (width*width + height3*height3)}" ixy="0.0" ixz="0.0"
-          iyy="${mass / 12.0 * (height3*height3 + width*width)}" iyz="0.0"
-          izz="${mass / 12.0 * (width*width + width*width)}"/>
-    </inertial>
-  </link>
-  <joint name="hokuyo_joint" type="fixed">
-    <axis xyz="0 1 0" />
-    <origin xyz="0 0 ${height3 - axel_offset/2}" rpy="0 0 0"/>
-    <parent link="link3"/>
-    <child link="hokuyo_link"/>
-  </joint>
-  Hokuyo Laser
-  <link name="hokuyo_link">
-    <collision>
-      <origin xyz="0 0 0" rpy="0 0 0"/>
-      <geometry>
-        <box size="0.1 0.1 0.1"/>
-      </geometry>
-    </collision>
-    <visual>
-      <origin xyz="0 0 0" rpy="0 0 0"/>
-      <geometry>
-        <mesh filename="package://amiro_description/meshes/hokuyo.dae"/>
-      </geometry>
-    </visual>
-    <inertial>
-      <mass value="1e-5" />
-      <origin xyz="0 0 0" rpy="0 0 0"/>
-      <inertia ixx="1e-6" ixy="0" ixz="0" iyy="1e-6" iyz="0" izz="1e-6" />
-    </inertial>
-  </link>
-  <joint name="camera_joint" type="fixed">
-    <axis xyz="0 1 0" />
-    <origin xyz="${camera_link} 0 ${height3 - axel_offset*2}" rpy="0 0 0"/>
-    <parent link="link3"/>
-    <child link="camera_link"/>
-  </joint>
-  <link name="camera_link">
-    <collision>
-      <origin xyz="0 0 0" rpy="0 0 0"/>
-      <geometry>
-        <box size="${camera_link} ${camera_link} ${camera_link}"/>
-      </geometry>
-    </collision>
-    <visual>
-      <origin xyz="0 0 0" rpy="0 0 0"/>
-      <geometry>
-        <box size="${camera_link} ${camera_link} ${camera_link}"/>
-      </geometry>
-      <material name="red"/>
-    </visual>
-    <inertial>
-      <mass value="1e-5" />
-      <origin xyz="0 0 0" rpy="0 0 0"/>
-      <inertia ixx="1e-6" ixy="0" ixz="0" iyy="1e-6" iyz="0" izz="1e-6" />
-    </inertial>
-  </link>
-  <transmission name="tran1">
-    <type>transmission_interface/SimpleTransmission</type>
-    <joint name="joint1">
-      <hardwareInterface>EffortJointInterface</hardwareInterface>
-    </joint>
-    <actuator name="motor1">
-      <hardwareInterface>EffortJointInterface</hardwareInterface>
-      <mechanicalReduction>1</mechanicalReduction>
-    </actuator>
-  </transmission>
-  <transmission name="tran2">
-    <type>transmission_interface/SimpleTransmission</type>
-    <joint name="joint2">
-      <hardwareInterface>EffortJointInterface</hardwareInterface>
-    </joint>
-    <actuator name="motor2">
-      <hardwareInterface>EffortJointInterface</hardwareInterface>
-      <mechanicalReduction>1</mechanicalReduction>
-    </actuator>
-  </transmission>-->
 </robot>

Commit message: Cleanup and usage of calculations for all parameters
Signed-off-by: Timo Korthals <tkorthals@cit-ec.uni-bielefeld.de>

File: amiro_description/urdf/amiro.xacro (robot description, xacro)
@@ -4,22 +4,38 @@
   <!-- Constants for robot dimensions -->
   <xacro:property name="PI" value="3.1415926535897931"/>
-  <xacro:property name="mass" value="0.4" /> <!-- amiro base mass -->
-  <xacro:property name="radius" value="0.05" /> <!-- amiro base radius -->
-  <xacro:property name="height" value="0.08" /> <!-- amiro base height -->
-  <xacro:property name="wheel_radius" value="0.03" /> <!-- amiro wheel radius -->
-  <xacro:property name="wheel_height" value="0.01" /> <!-- amiro wheel height -->
-  <xacro:property name="wheel_sep" value="0.069" /> <!-- amiro wheel seperation -->
-  <xacro:property name="wheel_dia" value="0.05571" /> <!-- amiro wheel diameter -->
-  <xacro:property name="wheel_mass" value="0.02" /> <!-- amiro wheel diameter -->
-  <xacro:property name="base_link_clearance" value="0.0026" /> <!-- space between floor and amiro base -->
-  <xacro:property name="base_link_height" value="${base_link_clearance + height / 2}" /> <!-- amiro base link height -->
-  <xacro:property name="prefix" value="" /> <!--""-->
-  <xacro:property name="base_link" value="${prefix}base_link" /> <!-- amiro base link -->
-  <xacro:property name="left_wheel_link" value="${prefix}left_wheel_link" /> <!-- amiro wheel link -->
-  <xacro:property name="right_wheel_link" value="${prefix}right_wheel_link" /> <!-- amiro wheel link -->
-  <xacro:property name="right_wheel_joint" value="${prefix}right_wheel_joint" /> <!-- amiro wheel joint -->
-  <xacro:property name="left_wheel_joint" value="${prefix}left_wheel_joint" /> <!-- amiro wheel joint -->
-  <xacro:property name="odom" value="${prefix}odom" /> <!-- amiro odometry topic/tf -->
-  <xacro:property name="cmd_vel" value="${prefix}cmd_vel" /> <!-- amiro differential command  topic -->
+  <xacro:property name="base_mass" value="0.4" /> <!-- (kg) base mass -->
+  <xacro:property name="base_diameter" value="0.099" /> <!-- (m) base diameter -->
+  <xacro:property name="base_radius" value="${base_diameter / 2}" /> <!-- (m) base radius -->
+  <xacro:property name="base_height" value="0.084" /> <!-- (m) base height from bottom of DiWheelDrive + extension + lid -->
+  <xacro:property name="base_clearance" value="0.01" /> <!-- (m) space between floor and base -->
+  <xacro:property name="wheel_height" value="0.006" /> <!-- (m) wheel height -->
+  <xacro:property name="wheel_sep" value="0.069" /> <!-- (m) wheel seperation -->
+  <xacro:property name="wheel_dia" value="0.05571" /> <!-- (m) wheel diameter -->
+  <xacro:property name="wheel_radius" value="${wheel_dia / 2}" /> <!-- (m) wheel radius -->
+  <xacro:property name="wheel_mass" value="0.02" /> <!-- (kg) wheel mass -->
+  <xacro:property name="wheel_damping" value="0.1" /> <!-- (?) wheel damping -->
+  <xacro:property name="caster_mass" value="0.01" /> <!-- (kg) caster mass -->
+  <xacro:property name="caster_dia" value="0.005" /> <!-- (m) caster diameter -->
+  <xacro:property name="caster_radius" value="${caster_dia / 2}" /> <!-- (m) caster radius -->
+  <xacro:property name="caster_clearance" value="0.001" /> <!-- (m) caster clearance above ground (needed, so that the robot is movable) -->
+  <xacro:property name="caster_sep" value="0.072" /> <!-- (m) caster seperation (we assume that there are two symetric caster in the front and back) -->
+  <!-- Constant dependent parameters -->
+  <xacro:property name="base_link_height" value="${base_clearance + base_height / 2}" /> <!-- base link height -->
+  <xacro:property name="caster_link_height" value="${caster_clearance + caster_radius}" /> <!-- caster link height -->
+  <!-- http://en.wikipedia.org/wiki/List_of_moment_of_inertia_tensors -->
+  <xacro:property name="base_ixx" value="${1/12 * base_mass * (3*base_radius*base_radius+base_height*base_height)}" />
+  <xacro:property name="base_iyy" value="${base_ixx}" />
+  <xacro:property name="base_izz" value="${1/2*base_mass*base_radius*base_radius}" />
+  <xacro:property name="wheel_ixx" value="${1/12 * wheel_mass * (3*wheel_radius*wheel_radius+wheel_height*wheel_height)}" />
+  <xacro:property name="wheel_iyy" value="${wheel_ixx}" />
+  <xacro:property name="wheel_izz" value="${1/2*wheel_mass*wheel_radius*wheel_radius}" />
+  <!-- Link, topic and other names -->
+  <xacro:property name="base_link" value="base_link" /> <!-- base link -->
+  <xacro:property name="left_wheel_link" value="left_wheel_link" /> <!-- wheel link -->
+  <xacro:property name="right_wheel_link" value="right_wheel_link" /> <!-- wheel link -->
+  <xacro:property name="right_wheel_joint" value="right_wheel_joint" /> <!-- wheel joint -->
+  <xacro:property name="left_wheel_joint" value="left_wheel_joint" /> <!-- wheel joint -->
+  <xacro:property name="odom" value="odom" /> <!-- odometry topic/tf -->
+  <xacro:property name="cmd_vel" value="cmd_vel" /> <!-- differential command  topic -->
   <xacro:property name="update_rate" value="$(arg update_rate)" /> <!-- update rate for the plugins and TFs -->
   <!-- Import all Gazebo-customization elements, including Gazebo colors -->
@@ -33,5 +49,5 @@
       <origin xyz="0 0 ${base_link_height}" rpy="0 0 0"/>
       <geometry>
-        <cylinder length="${height}" radius="${radius}"/>
+        <cylinder length="${base_height}" radius="${base_radius}"/>
       </geometry>
     </collision>
@@ -39,5 +55,5 @@
       <origin xyz="0 0 ${base_link_height}" rpy="0 0 0"/>
       <geometry>
-        <cylinder length="${height}" radius="${radius}"/>
+        <cylinder length="${base_height}" radius="${base_radius}"/>
       </geometry>
       <material name="orange"/>
@@ -45,45 +61,45 @@
     <inertial name='base_inertia'>
       <origin xyz="0 0 ${base_link_height}" rpy="0 0 0"/>
-      <mass value="${mass}"/>
+      <mass value="${base_mass}"/>
       <inertia
-        ixx="0.0012" ixy="0.0" ixz="0.0"
-        iyy="0.0012" iyz="0.0"
-        izz="0.005"/>
+        ixx="${base_ixx}" ixy="0.0" ixz="0.0"
+        iyy="${base_iyy}" iyz="0.0"
+        izz="${base_izz}"/>
     </inertial>
     <!-- Front caster -->
     <collision name='caster_front_collision'>
-      <origin xyz="0.042 0 0.001" rpy="0 0 0"/>
+      <origin xyz="${caster_sep / 2} 0 ${caster_link_height}" rpy="0 0 0"/>
       <geometry>
-        <sphere radius="0.002"/>
+        <sphere radius="${caster_radius}"/>
       </geometry>
     </collision>
     <visual name='caster_front_visual'>
-      <origin xyz="0.042 0 0.001" rpy="0 0 0"/>
+      <origin xyz="${caster_sep / 2} 0 ${caster_link_height}" rpy="0 0 0"/>
       <geometry>
-        <sphere radius="0.002"/>
+        <sphere radius="${caster_radius}"/>
       </geometry>
       <material name="orange"/>
     </visual>
     <inertial name='caster_front_inertia'>
-      <origin xyz="0.042 0 0.001" rpy="0 0 0"/>
-      <mass value="0.01"/>
+      <origin xyz="${caster_sep / 2} 0 ${caster_link_height}" rpy="0 0 0"/>
+      <mass value="${caster_mass}"/>
     </inertial>
     <!-- Back caster -->
     <collision name='caster_back_collision'>
-      <origin xyz="-0.042 0 0.001" rpy="0 0 0"/>
+      <origin xyz="-${caster_sep / 2} 0 ${caster_link_height}" rpy="0 0 0"/>
       <geometry>
-        <sphere radius="0.002"/>
+        <sphere radius="${caster_radius}"/>
       </geometry>
     </collision>
     <visual name='caster_back_visual'>
-      <origin xyz="-0.042 0 0.001" rpy="0 0 0"/>
+      <origin xyz="-${caster_sep / 2} 0 ${caster_link_height}" rpy="0 0 0"/>
       <geometry>
-        <sphere radius="0.002"/>
+        <sphere radius="${caster_radius}"/>
       </geometry>
       <material name="orange"/>
     </visual>
     <inertial name='caster_back_inertia'>
-      <origin xyz="-0.042 0 0.001" rpy="0 0 0"/>
-      <mass value="0.01"/>
+      <origin xyz="-${caster_sep / 2} 0 ${caster_link_height}" rpy="0 0 0"/>
+      <mass value="${caster_mass}"/>
     </inertial>
   </link>
@@ -92,7 +108,7 @@
     <parent link="${base_link}"/>
     <child link="${left_wheel_link}"/>
-    <origin xyz="0 ${wheel_radius} 0.02" rpy="0 ${PI/2} ${PI/2}"/>
+    <origin xyz="0 ${wheel_sep / 2} ${wheel_radius}" rpy="0 ${PI/2} ${PI/2}"/>
     <axis xyz="0 0 1"/>
-    <dynamics damping="0.1"/>
+    <dynamics damping="${wheel_damping}"/>
   </joint>
   <link name="${left_wheel_link}">
@@ -111,10 +127,10 @@
     </visual>
     <inertial>
-      <cylinder length="0.01" radius="0.03"/>
+      <cylinder length="${wheel_height}" radius="${wheel_radius}"/>
       <mass value="${wheel_mass}"/>
       <inertia
-        ixx="0.0000068453" ixy="0.0" ixz="0.0"
-        iyy="0.0000068453" iyz="0.0"
-        izz="0.0000075625"/>
+        ixx="${wheel_ixx}" ixy="0.0" ixz="0.0"
+        iyy="${wheel_iyy}" iyz="0.0"
+        izz="${wheel_izz}"/>
     </inertial>
   </link>
@@ -123,7 +139,7 @@
     <parent link="${base_link}"/>
     <child link="${right_wheel_link}"/>
-    <origin xyz="0 -${wheel_radius} 0.02" rpy="0 ${PI/2} ${PI/2}"/>
+    <origin xyz="0 -${wheel_sep / 2} ${wheel_radius}" rpy="0 ${PI/2} ${PI/2}"/>
     <axis xyz="0 0 1"/>
-    <dynamics damping="0.1"/>
+    <dynamics damping="${wheel_damping}"/>
   </joint>
   <link name="${right_wheel_link}">
@@ -142,10 +158,10 @@
     </visual>
     <inertial>
-      <cylinder length="0.01" radius="0.03"/>
+      <cylinder length="${wheel_height}" radius="${wheel_radius}"/>
       <mass value="${wheel_mass}"/>
       <inertia
-        ixx="0.0000068453" ixy="0.0" ixz="0.0"
-        iyy="0.0000068453" iyz="0.0"
-        izz="0.0000075625"/>
+        ixx="${wheel_ixx}" ixy="0.0" ixz="0.0"
+        iyy="${wheel_iyy}" iyz="0.0"
+        izz="${wheel_izz}"/>
     </inertial>
   </link>

Commit message: Add camera and laser models of AMiRo
Signed-off-by: Timo Korthals <tkorthals@cit-ec.uni-bielefeld.de>

File: amiro_description/urdf/amiro.xacro (robot description, xacro)
@@ -1,4 +1,3 @@
 <?xml version="1.0"?>
-<!-- Revolute-Revolute Manipulator -->
 <robot name="amiro" xmlns:xacro="http://www.ros.org/wiki/xacro">
   <!-- Constants for robot dimensions -->
@@ -23,4 +22,7 @@
   <xacro:property name="base_link_height" value="${base_clearance + base_height / 2}" /> <!-- base link height -->
   <xacro:property name="caster_link_height" value="${caster_clearance + caster_radius}" /> <!-- caster link height -->
+  <xacro:property name="lid_link_height" value="${base_clearance + base_height}" /> <!-- top of lid from base_link -->
+  <xacro:property name="camera_link_height" value="${base_clearance + 0.032}" /> <!-- camera height from base_link -->
+  <xacro:property name="camera_link_depth" value="${base_radius}" /> <!-- camera height from base_link -->
   <!-- http://en.wikipedia.org/wiki/List_of_moment_of_inertia_tensors -->
   <xacro:property name="base_ixx" value="${1/12 * base_mass * (3*base_radius*base_radius+base_height*base_height)}" />
