Commit message: Replace rigid caster slider by omnidirectional spheres to get rid of bumpy behaviour. Increase tourque to let the AMiRo drive faster (little tourque could cause numerical problems when reaching high velocities) Add more info to the README.md, also the fact the friction is a lie.
Signed-off-by: Timo Korthals <tkorthals@cit-ec.uni-bielefeld.de>

File: amiro_description/urdf/amiro.xacro (robot description, xacro)
@@ -32,4 +32,5 @@
   <xacro:property name="wheel_iyy" value="${wheel_ixx}" />
   <xacro:property name="wheel_izz" value="${1/2*wheel_mass*wheel_radius*wheel_radius}" />
+  <xacro:property name="caster_i" value="${2/5*caster_mass*caster_radius*caster_radius}" />
   <!-- Link, topic and other names -->
   <xacro:property name="base_link" value="base_link" /> <!-- base link -->
@@ -69,7 +70,17 @@
         izz="${base_izz}"/>
     </inertial>
-    <!-- Front caster -->
+  </link>
+  <!-- Front caster joint -->
+  <joint name="front_caster_joint" type="continuous">
+    <parent link="${base_link}"/>
+    <child link="front_caster_link"/>
+    <origin xyz="${caster_sep / 2} 0 ${caster_link_height}" rpy="0 0 0"/>
+    <axis xyz="1 1 1"/>
+    <dynamics damping="0.0"/>
+  </joint>
+  <!-- Front caster link -->
+  <link name="front_caster_link">
     <collision name='caster_front_collision'>
-      <origin xyz="${caster_sep / 2} 0 ${caster_link_height}" rpy="0 0 0"/>
+      <origin xyz="0 0 0" rpy="0 0 0"/>
       <geometry>
         <sphere radius="${caster_radius}"/>
@@ -77,5 +88,5 @@
     </collision>
     <visual name='caster_front_visual'>
-      <origin xyz="${caster_sep / 2} 0 ${caster_link_height}" rpy="0 0 0"/>
+      <origin xyz="0 0 0" rpy="0 0 0"/>
       <geometry>
         <sphere radius="${caster_radius}"/>
@@ -84,10 +95,24 @@
     </visual>
     <inertial name='caster_front_inertia'>
-      <origin xyz="${caster_sep / 2} 0 ${caster_link_height}" rpy="0 0 0"/>
+      <origin xyz="0 0 0" rpy="0 0 0"/>
+       <inertia
+        ixx="${caster_i}" ixy="0.0" ixz="0.0"
+        iyy="${caster_i}" iyz="0.0"
+        izz="${caster_i}"/>
       <mass value="${caster_mass}"/>
     </inertial>
-    <!-- Back caster -->
+  </link>
+  <!-- Back caster joint -->
+  <joint name="back_caster_joint" type="continuous">
+    <parent link="${base_link}"/>
+    <child link="back_caster_link"/>
+    <origin xyz="-${caster_sep / 2} 0 ${caster_link_height}" rpy="0 0 0"/>
+    <axis xyz="1 1 1"/>
+    <dynamics damping="0.0"/>
+  </joint>
+  <!-- Back caster link -->
+  <link name="back_caster_link">
     <collision name='caster_back_collision'>
-      <origin xyz="-${caster_sep / 2} 0 ${caster_link_height}" rpy="0 0 0"/>
+      <origin xyz="0 0 0" rpy="0 0 0"/>
       <geometry>
         <sphere radius="${caster_radius}"/>
@@ -95,5 +120,5 @@
     </collision>
     <visual name='caster_back_visual'>
-      <origin xyz="-${caster_sep / 2} 0 ${caster_link_height}" rpy="0 0 0"/>
+      <origin xyz="0 0 0" rpy="0 0 0"/>
       <geometry>
         <sphere radius="${caster_radius}"/>
@@ -102,5 +127,9 @@
     </visual>
     <inertial name='caster_back_inertia'>
-      <origin xyz="-${caster_sep / 2} 0 ${caster_link_height}" rpy="0 0 0"/>
+      <origin xyz="0 0 0" rpy="0 0 0"/>
+       <inertia
+        ixx="${caster_i}" ixy="0.0" ixz="0.0"
+        iyy="${caster_i}" iyz="0.0"
+        izz="${caster_i}"/>
       <mass value="${caster_mass}"/>
     </inertial>

Commit message: Add proximity sensors Add assembly_line world for lecture and projects
Signed-off-by: Timo Korthals <tkorthals@cit-ec.uni-bielefeld.de>

File: amiro_description/urdf/amiro.xacro (robot description, xacro)
@@ -3,4 +3,6 @@
   <!-- Constants for robot dimensions -->
   <xacro:property name="PI" value="3.1415926535897931"/>
+  <xacro:property name="PI_2" value="${PI / 2}"/>
+  <xacro:property name="deg2rad" value="${PI / 180}"/>
   <xacro:property name="base_mass" value="0.4" /> <!-- (kg) base mass -->
   <xacro:property name="base_diameter" value="0.099" /> <!-- (m) base diameter -->
@@ -25,4 +27,38 @@
   <xacro:property name="camera_link_height" value="${base_clearance + 0.032}" /> <!-- camera height from base_link -->
   <xacro:property name="camera_link_depth" value="${base_radius}" /> <!-- camera height from base_link -->
+  <xacro:property name="proximity_floor_z" value="${base_clearance}" /> <!-- Proximity floor sensor over ground -->
+  <xacro:property name="proximity_floor_x_0" value="${base_radius - 0.005}" />
+  <xacro:property name="proximity_floor_y_0" value="-0.0035" />
+  <xacro:property name="proximity_floor_x_1" value="${base_radius - 0.021}" />
+  <xacro:property name="proximity_floor_y_1" value="-0.032" />
+  <xacro:property name="proximity_floor_x_2" value="${base_radius - 0.021}" />
+  <xacro:property name="proximity_floor_y_2" value="0.032" />
+  <xacro:property name="proximity_floor_x_3" value="${base_radius - 0.005}" />
+  <xacro:property name="proximity_floor_y_3" value="0.0035" />
+  <xacro:property name="proximity_ring_z" value="${0.027 + base_clearance}" /> <!-- Proximity ring sensor over ground -->
+  <xacro:property name="proximity_ring_yaw_3" value="${ 22.5 * deg2rad}" />
+  <xacro:property name="proximity_ring_yaw_2" value="${ 67.5 * deg2rad}" />
+  <xacro:property name="proximity_ring_yaw_1" value="${112.5 * deg2rad}" />
+  <xacro:property name="proximity_ring_yaw_0" value="${157.5 * deg2rad}" />
+  <xacro:property name="proximity_ring_yaw_7" value="${202.5 * deg2rad}" />
+  <xacro:property name="proximity_ring_yaw_6" value="${247.5 * deg2rad}" />
+  <xacro:property name="proximity_ring_yaw_5" value="${292.5 * deg2rad}" />
+  <xacro:property name="proximity_ring_yaw_4" value="${337.5 * deg2rad}" />
+  <xacro:property name="proximity_ring_x_0" value="${base_radius * cos(proximity_ring_yaw_0)}" />
+  <xacro:property name="proximity_ring_y_0" value="${base_radius * sin(proximity_ring_yaw_0)}" />
+  <xacro:property name="proximity_ring_x_1" value="${base_radius * cos(proximity_ring_yaw_1)}" />
+  <xacro:property name="proximity_ring_y_1" value="${base_radius * sin(proximity_ring_yaw_1)}" />
+  <xacro:property name="proximity_ring_x_2" value="${base_radius * cos(proximity_ring_yaw_2)}" />
+  <xacro:property name="proximity_ring_y_2" value="${base_radius * sin(proximity_ring_yaw_2)}" />
+  <xacro:property name="proximity_ring_x_3" value="${base_radius * cos(proximity_ring_yaw_3)}" />
+  <xacro:property name="proximity_ring_y_3" value="${base_radius * sin(proximity_ring_yaw_3)}" />
+  <xacro:property name="proximity_ring_x_4" value="${base_radius * cos(proximity_ring_yaw_4)}" />
+  <xacro:property name="proximity_ring_y_4" value="${base_radius * sin(proximity_ring_yaw_4)}" />
+  <xacro:property name="proximity_ring_x_5" value="${base_radius * cos(proximity_ring_yaw_5)}" />
+  <xacro:property name="proximity_ring_y_5" value="${base_radius * sin(proximity_ring_yaw_5)}" />
+  <xacro:property name="proximity_ring_x_6" value="${base_radius * cos(proximity_ring_yaw_6)}" />
+  <xacro:property name="proximity_ring_y_6" value="${base_radius * sin(proximity_ring_yaw_6)}" />
+  <xacro:property name="proximity_ring_x_7" value="${base_radius * cos(proximity_ring_yaw_7)}" />
+  <xacro:property name="proximity_ring_y_7" value="${base_radius * sin(proximity_ring_yaw_7)}" />
   <!-- http://en.wikipedia.org/wiki/List_of_moment_of_inertia_tensors -->
   <xacro:property name="base_ixx" value="${1/12 * base_mass * (3*base_radius*base_radius+base_height*base_height)}" />

Commit message: amiro_description: Add meshes of extended AMiRo and wheels                    Add viz. of meshes (TODO: Textures are missing) amiro_gazebo: Cleanup and fix for gazebo/standalone launch amiro_description/urdf/camera/astra.xacro: Fix namespace
Signed-off-by: Timo Korthals <tkorthals@cit-ec.uni-bielefeld.de>

File: amiro_description/urdf/amiro.xacro (robot description, xacro)
@@ -21,4 +21,8 @@
   <xacro:property name="caster_clearance" value="0.001" /> <!-- (m) caster clearance above ground (needed, so that the robot is movable) -->
   <xacro:property name="caster_sep" value="0.072" /> <!-- (m) caster seperation (we assume that there are two symetric caster in the front and back) -->
+  <!-- Use CAD mesh model or the primitive one -->
+  <xacro:property name="use_mesh_model" value="true"/>
+  <xacro:property name="mesh_scale" value="0.0254"/>
+  <xacro:property name="mesh_clearance" value="${base_clearance + 0.002}" />
   <!-- Constant dependent parameters -->
   <xacro:property name="base_link_height" value="${base_clearance + base_height / 2}" /> <!-- base link height -->
@@ -78,8 +82,8 @@
   <xacro:property name="cmd_vel" value="cmd_vel" /> <!-- differential command  topic -->
   <xacro:property name="update_rate" value="$(arg update_rate)" /> <!-- update rate for the plugins and TFs -->
+  <!-- Import Rviz colors -->
+  <xacro:include filename="$(find amiro_description)/urdf/materials.xacro" />
   <!-- Import all Gazebo-customization elements, including Gazebo colors -->
   <xacro:include filename="$(find amiro_description)/urdf/amiro.gazebo" />
-  <!-- Import Rviz colors -->
-  <xacro:include filename="$(find amiro_description)/urdf/materials.xacro" />
   <!-- Base Link -->
   <link name="${base_link}">
@@ -92,10 +96,33 @@
     </collision>
     <visual name='base_visual'>
-      <origin xyz="0 0 ${base_link_height}" rpy="0 0 0"/>
-      <geometry>
-        <cylinder length="${base_height}" radius="${base_radius}"/>
-      </geometry>
-      <material name="orange"/>
+      <xacro:if value="${use_mesh_model == 'true'}">
+        <origin xyz="${base_radius} -${base_radius} ${mesh_clearance}" rpy="0 0 ${PI/2}"/>
+        <geometry>
+<!--         <mesh filename="package://amiro_description/meshes/laser/hokuyo.dae"/> -->
+<!--           <mesh filename="package://amiro_description/meshes/robot/WheelDrive_degenerateDissolve_cleanUpGeometry002.dae"/> -->
+<!--         <mesh filename="package://amiro_description/meshes/robot/BaseAmiroOnly_degenerateDissolve_cleanUpGeometry005.dae" scale="${mesh_scale} ${mesh_scale} ${mesh_scale}"/> -->
+        <mesh filename="package://amiro_description/meshes/robot/ExtendedAmiroOnly_degenerateDissolve_cleanUpGeometry005.dae" scale="${mesh_scale} ${mesh_scale} ${mesh_scale}"/>
+<!--         <mesh filename="package://amiro_description/meshes/robot/ExtendedAmiro_degenerateDissolve_cleanUpGeometry004.dae"/> -->
+        </geometry>
+      </xacro:if>
+      <xacro:if value="${use_mesh_model != 'true'}">
+        <origin xyz="0 0 ${base_link_height}" rpy="0 0 0"/>
+        <geometry>
+          <cylinder length="${base_height}" radius="${base_radius}"/>
+        </geometry>
+        <material name="orange"/>
+      </xacro:if>
     </visual>
+  </link>
+  <!-- Dummy joint, so that the root link has no inertia -->
+  <joint name="base_inertia_joint" type="fixed">
+    <parent link="${base_link}"/>
+    <child link="base_inertia_link"/>
+    <origin xyz="0 0 0" rpy="0 0 0"/>
+    <axis xyz="1 1 1"/>
+    <dynamics damping="0.0"/>
+  </joint>
+  <!-- Dummy link, so that the root link has no inertia -->
+  <link name="base_inertia_link">
     <inertial name='base_inertia'>
       <origin xyz="0 0 ${base_link_height}" rpy="0 0 0"/>
@@ -123,11 +150,13 @@
       </geometry>
     </collision>
-    <visual name='caster_front_visual'>
-      <origin xyz="0 0 0" rpy="0 0 0"/>
-      <geometry>
-        <sphere radius="${caster_radius}"/>
-      </geometry>
-      <material name="orange"/>
-    </visual>
+    <xacro:if value="${use_mesh_model != 'true'}">
+      <visual name='caster_front_visual'>
+        <origin xyz="0 0 0" rpy="0 0 0"/>
+        <geometry>
+          <sphere radius="${caster_radius}"/>
+        </geometry>
+        <material name="orange"/>
+      </visual>
+    </xacro:if>
     <inertial name='caster_front_inertia'>
       <origin xyz="0 0 0" rpy="0 0 0"/>
@@ -155,11 +184,13 @@
       </geometry>
     </collision>
-    <visual name='caster_back_visual'>
-      <origin xyz="0 0 0" rpy="0 0 0"/>
-      <geometry>
-        <sphere radius="${caster_radius}"/>
-      </geometry>
-      <material name="orange"/>
-    </visual>
+    <xacro:if value="${use_mesh_model != 'true'}">
+      <visual name='caster_back_visual'>
+        <origin xyz="0 0 0" rpy="0 0 0"/>
+        <geometry>
+          <sphere radius="${caster_radius}"/>
+        </geometry>
+        <material name="orange"/>
+      </visual>
+    </xacro:if>
     <inertial name='caster_back_inertia'>
       <origin xyz="0 0 0" rpy="0 0 0"/>
@@ -187,9 +218,17 @@
     </collision>
     <visual>
-      <cylinder length="${wheel_height}" radius="${wheel_radius}"/>
-      <geometry>
-        <cylinder length="${wheel_height}" radius="${wheel_radius}"/>
-      </geometry>
-      <material name="black"/>
+      <xacro:if value="${use_mesh_model == 'true'}">
+        <origin xyz="0 0 0" rpy="${PI/2} 0 0"/>
+        <geometry>
+          <mesh filename="package://amiro_description/meshes/robot/WheelDrive_degenerateDissolve_cleanUpGeometry002_centered.dae" scale="${mesh_scale} ${mesh_scale} ${mesh_scale}"/>
+        </geometry>
+      </xacro:if>
+      <xacro:if value="${use_mesh_model != 'true'}">
+        <cylinder length="${wheel_height}" radius="${wheel_radius}"/>
+        <geometry>
+          <cylinder length="${wheel_height}" radius="${wheel_radius}"/>
+        </geometry>
+        <material name="black"/>
+      </xacro:if>
     </visual>
     <inertial>
@@ -218,9 +257,18 @@
     </collision>
     <visual>
-      <cylinder length="${wheel_height}" radius="${wheel_radius}"/>
-      <geometry>
-        <cylinder length="${wheel_height}" radius="${wheel_radius}"/>
-      </geometry>
-      <material name="black"/>
+      <xacro:if value="${use_mesh_model == 'true'}">
+<!--         <origin xyz="0 -${wheel_sep / 2} ${wheel_radius + 0.005}" rpy="0 0 0"/> -->
+        <origin xyz="0 0 0" rpy="${PI/2} 0 0"/>
+        <geometry>
+          <mesh filename="package://amiro_description/meshes/robot/WheelDrive_degenerateDissolve_cleanUpGeometry002_centered.dae" scale="${mesh_scale} ${mesh_scale} ${mesh_scale}"/>
+        </geometry>
+      </xacro:if>
+      <xacro:if value="${use_mesh_model != 'true'}">
+        <cylinder length="${wheel_height}" radius="${wheel_radius}"/>
+        <geometry>
+          <cylinder length="${wheel_height}" radius="${wheel_radius}"/>
+        </geometry>
+        <material name="black"/>
+      </xacro:if>
     </visual>
     <inertial>

Commit message: Fix missing tf for caster wheels and add more examples in amiro_world.launch
Signed-off-by: Timo Korthals <tkorthals@cit-ec.uni-bielefeld.de>

File: amiro_description/urdf/amiro.xacro (robot description, xacro)
@@ -22,7 +22,15 @@
   <xacro:property name="caster_sep" value="0.072" /> <!-- (m) caster seperation (we assume that there are two symetric caster in the front and back) -->
   <!-- Use CAD mesh model or the primitive one -->
-  <xacro:property name="use_mesh_model" value="true"/>
+  <xacro:property name="use_mesh_model" value="$(arg use_mesh_model)"/>
   <xacro:property name="mesh_scale" value="0.0254"/>
   <xacro:property name="mesh_clearance" value="${base_clearance + 0.002}" />
+  <!-- Decide if the joints are controlled by Gazebo or just fixed if Gazebo is not used -->
+  <xacro:property name="use_gazebo" value="$(arg use_gazebo)"/>
+  <xacro:if value="${use_gazebo == 'true'}">
+    <xacro:property name="joint_types" value="continuous"/>
+  </xacro:if>
+  <xacro:if value="${use_gazebo != 'true'}">
+    <xacro:property name="joint_types" value="fixed"/>
+  </xacro:if>
   <!-- Constant dependent parameters -->
   <xacro:property name="base_link_height" value="${base_clearance + base_height / 2}" /> <!-- base link height -->
@@ -100,8 +108,8 @@
         <geometry>
 <!--         <mesh filename="package://amiro_description/meshes/laser/hokuyo.dae"/> -->
-<!--           <mesh filename="package://amiro_description/meshes/robot/WheelDrive_degenerateDissolve_cleanUpGeometry002.dae"/> -->
+<!--         <mesh filename="package://amiro_description/meshes/robot/WheelDrive_degenerateDissolve_cleanUpGeometry002.dae"/> -->
+<!--         <mesh filename="package://amiro_description/meshes/robot/ExtendedAmiro_degenerateDissolve_cleanUpGeometry004.dae"/> -->
 <!--         <mesh filename="package://amiro_description/meshes/robot/BaseAmiroOnly_degenerateDissolve_cleanUpGeometry005.dae" scale="${mesh_scale} ${mesh_scale} ${mesh_scale}"/> -->
         <mesh filename="package://amiro_description/meshes/robot/ExtendedAmiroOnly_degenerateDissolve_cleanUpGeometry005.dae" scale="${mesh_scale} ${mesh_scale} ${mesh_scale}"/>
-<!--         <mesh filename="package://amiro_description/meshes/robot/ExtendedAmiro_degenerateDissolve_cleanUpGeometry004.dae"/> -->
         </geometry>
       </xacro:if>
@@ -135,5 +143,5 @@
   </link>
   <!-- Front caster joint -->
-  <joint name="front_caster_joint" type="continuous">
+  <joint name="front_caster_joint" type="fixed">
     <parent link="${base_link}"/>
     <child link="front_caster_link"/>
@@ -169,5 +177,5 @@
   </link>
   <!-- Back caster joint -->
-  <joint name="back_caster_joint" type="continuous">
+  <joint name="back_caster_joint" type="fixed">
     <parent link="${base_link}"/>
     <child link="back_caster_link"/>
@@ -203,5 +211,5 @@
   </link>
   <!-- Left wheel -->
-  <joint name="${left_wheel_joint}" type="continuous">
+  <joint name="${left_wheel_joint}" type="${joint_types}">
     <parent link="${base_link}"/>
     <child link="${left_wheel_link}"/>
@@ -242,5 +250,5 @@
   </link>
   <!-- Right wheel -->
-  <joint name="${right_wheel_joint}" type="continuous">
+  <joint name="${right_wheel_joint}" type="${joint_types}">
     <parent link="${base_link}"/>
     <child link="${right_wheel_link}"/>
@@ -258,5 +266,4 @@
     <visual>
       <xacro:if value="${use_mesh_model == 'true'}">
-<!--         <origin xyz="0 -${wheel_sep / 2} ${wheel_radius + 0.005}" rpy="0 0 0"/> -->
         <origin xyz="0 0 0" rpy="${PI/2} 0 0"/>
         <geometry>

File: amiro_description/urdf/laser/hokuyo.xacro (robot description, xacro)
@@ -63,7 +63,4 @@
             <frameName>${name}</frameName>
           </plugin>
-          <!--
-          <plugin name="laser" filename="libRayPlugin.so" />
-          -->
           <always_on>1</always_on>
           <update_rate>10</update_rate>

Commit message: Change 'true'/'false' statements to 1/0 since melodic does not handle this well
Signed-off-by: Timo Korthals <tkorthals@cit-ec.uni-bielefeld.de>

File: amiro_description/urdf/amiro.xacro (robot description, xacro)
@@ -27,8 +27,8 @@
   <!-- Decide if the joints are controlled by Gazebo or just fixed if Gazebo is not used -->
   <xacro:property name="use_gazebo" value="$(arg use_gazebo)"/>
-  <xacro:if value="${use_gazebo == 'true'}">
+  <xacro:if value="${use_gazebo == 1}">
     <xacro:property name="joint_types" value="continuous"/>
   </xacro:if>
-  <xacro:if value="${use_gazebo != 'true'}">
+  <xacro:if value="${use_gazebo == 0}">
     <xacro:property name="joint_types" value="fixed"/>
   </xacro:if>
@@ -104,5 +104,5 @@
     </collision>
     <visual name='base_visual'>
-      <xacro:if value="${use_mesh_model == 'true'}">
+      <xacro:if value="${use_mesh_model == 1}">
         <origin xyz="${base_radius} -${base_radius} ${mesh_clearance}" rpy="0 0 ${PI/2}"/>
         <geometry>
@@ -111,8 +111,8 @@
 <!--         <mesh filename="package://amiro_description/meshes/robot/ExtendedAmiro_degenerateDissolve_cleanUpGeometry004.dae"/> -->
 <!--         <mesh filename="package://amiro_description/meshes/robot/BaseAmiroOnly_degenerateDissolve_cleanUpGeometry005.dae" scale="${mesh_scale} ${mesh_scale} ${mesh_scale}"/> -->
-        <mesh filename="package://amiro_description/meshes/robot/ExtendedAmiroOnly_degenerateDissolve_cleanUpGeometry005.dae" scale="${mesh_scale} ${mesh_scale} ${mesh_scale}"/>
-        </geometry>
-      </xacro:if>
-      <xacro:if value="${use_mesh_model != 'true'}">
+          <mesh filename="package://amiro_description/meshes/robot/ExtendedAmiroOnly_degenerateDissolve_cleanUpGeometry005.dae" scale="${mesh_scale} ${mesh_scale} ${mesh_scale}"/>
+        </geometry>
+      </xacro:if>
+      <xacro:if value="${use_mesh_model == 0}">
         <origin xyz="0 0 ${base_link_height}" rpy="0 0 0"/>
         <geometry>
@@ -158,5 +158,5 @@
       </geometry>
     </collision>
-    <xacro:if value="${use_mesh_model != 'true'}">
+    <xacro:if value="${use_mesh_model == 0}">
       <visual name='caster_front_visual'>
         <origin xyz="0 0 0" rpy="0 0 0"/>
@@ -192,5 +192,5 @@
       </geometry>
     </collision>
-    <xacro:if value="${use_mesh_model != 'true'}">
+    <xacro:if value="${use_mesh_model == 0}">
       <visual name='caster_back_visual'>
         <origin xyz="0 0 0" rpy="0 0 0"/>
@@ -226,5 +226,5 @@
     </collision>
     <visual>
-      <xacro:if value="${use_mesh_model == 'true'}">
+      <xacro:if value="${use_mesh_model == 1}">
         <origin xyz="0 0 0" rpy="${PI/2} 0 0"/>
         <geometry>
@@ -232,5 +232,5 @@
         </geometry>
       </xacro:if>
-      <xacro:if value="${use_mesh_model != 'true'}">
+      <xacro:if value="${use_mesh_model == 0}">
         <cylinder length="${wheel_height}" radius="${wheel_radius}"/>
         <geometry>
@@ -265,5 +265,5 @@
     </collision>
     <visual>
-      <xacro:if value="${use_mesh_model == 'true'}">
+      <xacro:if value="${use_mesh_model == 1}">
         <origin xyz="0 0 0" rpy="${PI/2} 0 0"/>
         <geometry>
@@ -271,5 +271,5 @@
         </geometry>
       </xacro:if>
-      <xacro:if value="${use_mesh_model != 'true'}">
+      <xacro:if value="${use_mesh_model == 0}">
         <cylinder length="${wheel_height}" radius="${wheel_radius}"/>
         <geometry>
