Commit message: Fix accumulated sum in proximity floor mockup sensors Add debug section to readme
Signed-off-by: Timo Korthals <tkorthals@cit-ec.uni-bielefeld.de>

File: amiro_description/urdf/proximity/floor.xacro (robot description, xacro)
@@ -18,5 +18,5 @@
       <inertia ixx="1e-6" ixy="0" ixz="0" iyy="1e-6" iyz="0" izz="1e-6" />
     </inertial>
-<!--    <visual>
+    <visual>
       <origin xyz="0 0 0" rpy="0 1.57 0"/>
       <geometry>
@@ -24,5 +24,5 @@
       </geometry>
       <material name="black"/>
-    </visual>-->
+    </visual>
     <collision>
       <origin xyz="0 0 0" rpy="0 1.57 0"/>
